File: hw/sci2can.sch (KiCad schematic (older format))
At the start: 34 parts, among them IC1 MC9S08DZ60xLC, J1 BDM, J2 Screw Terminal, Q1 4MHz, Q2 MGSF1N03L*, U1 uA7805, U2 PCA82C251

Commit message: hw 1v02
Parts:
- removed D2: POWER*, Diode_SMD:D_0603_1608Metric_Pad1.05x0.95mm_HandSolder, symbol Device:LED
- removed D4: STOUT*, Diode_SMD:D_0603_1608Metric_Pad1.05x0.95mm_HandSolder, symbol Device:LED
- removed R1: 680*, Resistor_SMD:R_0603_1608Metric_Pad1.05x0.95mm_HandSolder, symbol Device:R
- removed R13: 10k*, Resistor_SMD:R_0603_1608Metric_Pad1.05x0.95mm_HandSolder, symbol Device:R
- removed R14: 5k*, Resistor_SMD:R_0603_1608Metric_Pad1.05x0.95mm_HandSolder, symbol Device:R
- removed U1: uA7805, Package_TO_SOT_THT:TO-220-3_Horizontal_TabDown, symbol Regulator_Linear:uA7805
- added Cs2: 1uF, Capacitor_SMD:C_0603_1608Metric_Pad1.05x0.95mm_HandSolder, symbol Device:C
- added Cs3: 220pF, Capacitor_SMD:C_0603_1608Metric_Pad1.05x0.95mm_HandSolder, symbol Device:C
- added Cs6: 10uF, Capacitor_SMD:C_0603_1608Metric_Pad1.05x0.95mm_HandSolder, symbol Device:C
- added Di1: BZT52C4V7, Diode_SMD:D_SOD-123, symbol Device:D_Zener
- added Ds2: SMAJ33A 38.7V, Diode_SMD:D_SMA, symbol Device:D_Zener
- added Ds3: SS34, Diode_SMD:D_SMA, symbol Diode:B120-E3
- added Ls1: 47uH, Inductor_SMD:L_2816_7142Metric_Pad3.20x4.45mm_HandSolder, symbol pspice:INDUCTOR
- added Ri7, Rs5: 10k, Resistor_SMD:R_0603_1608Metric_Pad1.05x0.95mm_HandSolder, symbol Device:R
- added Ri8: 1k, Resistor_SMD:R_0603_1608Metric_Pad1.05x0.95mm_HandSolder, symbol Device:R
- added Ri9: ?*, Resistor_SMD:R_0603_1608Metric_Pad1.05x0.95mm_HandSolder, symbol Device:R
- added Rs3: 1M, Resistor_SMD:R_0603_1608Metric_Pad1.05x0.95mm_HandSolder, symbol Device:R
- added Rs4: 3k, Resistor_SMD:R_0603_1608Metric_Pad1.05x0.95mm_HandSolder, symbol Device:R
- added T1: TSM2308*, Package_TO_SOT_SMD:SOT-23, symbol Transistor_FET:TSM2302CX
- added U1: ME3116, Package_TO_SOT_SMD:SOT-23-6_Handsoldering, symbol butyi:ME3116
- Cs1: renamed from C1; value 1uF -> 10uF 50V; footprint Capacitor_SMD:C_0603_1608Metric_Pad1.05x0.95mm_HandSolder -> Capacitor_SMD:C_Elec_5x5.8; symbol Device:C -> Device:CP
- Cs4: renamed from C2; value 10nF -> 1uF
- Cs5: renamed from C3; value 1uF -> 10uF
- Di2: renamed from D5; value 4V7 -> BZT52C4V7; footprint Diode_SMD:D_1206_3216Metric_Pad1.42x1.75mm_HandSolder -> Diode_SMD:D_SOD-123
- J1: footprint Connector_PinHeader_2.54mm:PinHeader_2x03_P2.54mm_Vertical -> Connector_PinHeader_2.54mm:PinHeader_2x05_P2.54mm_Vertical; symbol Connector_Generic:Conn_02x03_Odd_Even -> Connector_Generic:Conn_02x05_Odd_Even
- Rb1: renamed from R10; value 10k* -> 10k
- Rc2: renamed from RT1; value 120 -> 100
- Ri4: renamed from R6; value Reserved* -> ?*
- Rl1: renamed from R12; value 680 -> 1k
- Rs1: renamed from R2; value 100k* -> 100k
- Rs2: renamed from R3; value 10k* -> 10k
- T2: renamed from Q2; value MGSF1N03L* -> TSM2308*; symbol Transistor_FET:BSS138 -> Transistor_FET:TSM2302CX
- renumbered C7 to Ci2, C4 to Cq1, C5 to Cq2, C6 to Cr1, D3 to Dl1, D1 to Ds1, R8 to Rc1, R7 to Ri1, R4 to Ri2, R5 to Ri3, R9 to Rq1, R11 to Rr1, IC1 to uC1
Connections:
- net OUT is gone; now on net IO2: J2.3 (Pin_3), T2.3 (D)
- net GND: now also Cs6.2, Di1.2 (A), Ds2.2 (A), Ds3.2 (A), Ri9.1, Rs4.2, T1.2 (S), U1.2 (GND)
- net RESET: now also Rr1.1; no longer Rr1.2
- net RXCAN: no longer J1.3 (Pin_3)
- net RxD1: now also J1.5 (Pin_5); no longer Di2.1 (K)
- net TXCAN: no longer J1.5 (Pin_5)
- net PTE3: now reaches uC1.10 (PTE3)
- net PTE3: now also J1.7 (Pin_7)
- net SCL: now reaches uC1.11 (PTE4)
- net SCL: now also J1.10 (Pin_10)
- net SDA: now reaches uC1.12 (PTE5)
- net SDA: now also J1.9 (Pin_9)
- net FET1: now reaches uC1.18 (PTD3)
- net FET1: now also T1.1 (G)
- net IN2: now reaches uC1.25 (PTA1)
- net IN2: now also Ri8.1, Ri9.2
- net TxD1: now reaches uC1.7 (PTE0)
- net TxD1: now also J1.3 (Pin_3)
- net PTE2: now reaches uC1.9 (PTE2)
- net PTE2: now also J1.8 (Pin_8)
- net at Cs1.1, Ds1.1 (K): now also Ds2.1 (K), Rs3.2, U1.5 (VIN)
- net at Ci2.1, Ri2.1, Ri3.2: now also Di2.1 (K)
- net +5V renamed +3V3
- net +3V3: now also Rr1.2, Cs3.2, Cs6.1, Ls1.2, Rs5.1; no longer Rr1.1
- net FET renamed FET2
- net IN renamed IO2
- net IO2: no longer J2.4 (Pin_4)
- new net: Cs2.1, U1.1 (BST)
- new net: Cs3.1, Rs4.1, Rs5.2, U1.3 (FB)
- new net: Rs3.1, U1.4 (EN)
- new net: Cs2.2, Ds3.1 (K), Ls1.1, U1.6 (SW)
- new net: Di1.1 (K), Ri7.1, Ri8.2
- new net IO1: J2.4 (Pin_4), Ri7.2, T1.3 (D)
- no-connect marks 19 -> 12
Other:
- note removed: "** When OSCILL_SUPP is enabled"
- note removed: "High during CAN Tx ISR **"
- note removed: "High during CAN Tx burst **"
- note removed: "High during RTC ISR **"
- note removed: "High during SCI Rx ISR **"
- note removed: "High during SCI Rx burst **"
- moved on the sheet: Ci2, Cs4, Cs5, Di2, Ds1, Rb1, Rc1, Rc2, Ri1, Ri2, Ri3, Ri4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

Commit message: HW SW update, 0.96 inch display
Parts:
- removed Ci2: 10nF, Capacitor_SMD:C_0603_1608Metric_Pad1.05x0.95mm_HandSolder, symbol Device:C
- removed Di1, Di2: BZT52C4V7, Diode_SMD:D_SOD-123, symbol Device:D_Zener
- removed Ds2: SMAJ33A 38.7V, Diode_SMD:D_SMA, symbol Device:D_Zener
- removed uC1: MC9S08DZ60xLC, Package_QFP:LQFP-32_7x7mm_P0.8mm, symbol MCU_NXP_S08:MC9S08DZ60xLC
- added Cs7: 1uF, Capacitor_SMD:C_0603_1608Metric_Pad1.05x0.95mm_HandSolder, symbol Device:C
- added Dc1, Dc2, Di1, Di2, Ds4: ESD5Z5V0, Diode_SMD:D_SOD-523, symbol butyi:ESD5Z5V0
- added Ds2: SMAJ33A, Diode_SMD:D_SMA, symbol butyi:SMAJ33A
- added Js1: Jumper, Jumper:SolderJumper-2_P1.3mm_Open_RoundedPad1.0x1.5mm, symbol Device:Jumper
- added Ui1: 74HC1G125GW, Package_TO_SOT_SMD:SOT-353_SC-70-5_Handsoldering, symbol butyi:74HC1G125GW
- added uC1: MC9S08DZ60xLF, Package_QFP:LQFP-48_7x7mm_P0.5mm, symbol MCU_NXP_S08:MC9S08DZ60xLF
- Cs6: value 10uF -> 100nF
- Ls1: value 47uH -> 10uH
- Ri3: value 1k -> 1k*
- Rs4: value 3k -> 2k
Connections:
- net BKGD: now also uC1.33 (BKGD/MS)
- net CANH: now also Dc2.1 (A1)
- net CANL: now also Dc1.1 (A1)
- net EXTAL: now also uC1.6 (PTG0/EXTAL)
- net FET1: now also uC1.26 (PTD3)
- net FET2: now also uC1.25 (PTD2)
- net GND: now also Cs7.1, Dc1.2 (A2), Dc2.2 (A2), Di1.2 (A2), Di2.2 (A2), Ds2.2 (A2), Ds4.2 (A2), Ui1.1 (!OE), Ui1.3 (GND), uC1.29 (VSS), uC1.42 (VSSA/VREFL), uC1.5 (VSS)
- net IN2: now also uC1.37 (PTA1)
- net LED2: now also uC1.48 (PTA6)
- net PTE2: now also uC1.13 (PTE2)
- net PTE3: now also uC1.14 (PTE3)
- net RESET: now also uC1.8 (~RESET)
- net RXCAN: now also uC1.22 (PTE7)
- net RxD1: now also uC1.12 (PTE1); no longer Ri3.1, Ri4.2
- net SCL: now also uC1.15 (PTE4)
- net SDA: now also uC1.16 (PTE5)
- net TXCAN: now also uC1.21 (PTE6)
- net TxD1: now also uC1.11 (PTE0)
- net UZ_MEAS: now also uC1.46 (PTA5)
- net XTAL: now also uC1.7 (PTG1/XTAL)
- net at Cs1.1, Ds1.1 (K), Rs3.2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: now also Ds2.1 (A1)
- net at Ri2.1, Ri3.2: now also Di2.1 (A1), Ui1.2 (IN)
- net at Ri7.1, Ri8.2: now also Di1.1 (A1)
- net +3V3: no longer names the net of Cs3.2, Cs5.1, Cs6.1, Ls1.2, Rs5.1
- net +3V3: now also Js1.1; no longer Cs4.1, J1.6 (Pin_6), Rb1.1, Rr1.2, U2.3 (VCC)
- new net +5V: Cs4.1, Cs7.2, Ds4.1 (A1), J1.6 (Pin_6), Js1.2, Rb1.1, Rr1.2, U2.3 (VCC), Ui1.5 (VCC), uC1.30 (VDD), uC1.4 (VDD), uC1.43 (VDDA/VREFH)
- new net RxD2: Ri3.1, Ri4.2, Ui1.4 (OUT), uC1.18 (PTF1), uC1.35 (PTA0)
- no-connect marks 12 -> 25
Other:
- moved on the sheet: Cs4, Cs6, Ri1, Ri2, Ri3, Ri4, Ri7, Ri8, Ri9
